File: circuit/LineFollowingRobotCircuit.brd (EAGLE design)
At the start: 259.3 x 146.3 mm, 14 parts, among them M1 MOTOR_DG01D, M2 MOTOR_DG01D, U1 ARDUINO-UNO-R3-SHIELD, U2 L293E, U3 74HC04_PDIP, U5 IR-RECEIVERTSOP48

Commit message: chore(circuit): added new circuit
Parts:
- removed D9: DIODEDIODE-AXIAL, Tinkercad:DIODE-AXIAL
- removed U5: IR-RECEIVERTSOP48, Tinkercad:TSOP48
- added D7: DIODEDIODE-AXIAL, Tinkercad:DIODE-AXIAL
- added PIR1, PIR2: PIR-SENSOR_28027, Tinkercad:28027
- U2: value L293E -> IR-RECEIVERTSOP48; device Tinkercad:DIP762W53P254L1969H508Q16B -> Tinkercad:TSOP48
- U3: value 74HC04_PDIP -> L293E; device Tinkercad:DIP762W53P254L1969H508Q14B -> Tinkercad:DIP762W53P254L1969H508Q16B
- moved M2 147.3 mm to (99.2, 74.3), turned to 0 degrees
- moved U2 111.2 mm to (110.0, 146.0), turned to 0 degrees
- moved D8 95.0 mm to (114.6, 65.5)
- moved D5 92.7 mm to (117.2, 90.9), turned to 360 degrees
- moved D6 89.9 mm to (117.2, 62.9)
- moved U3 69.1 mm to (133.7, 76.9)
- moved M1 52.6 mm to (176.8, 83.0), turned to 180 degrees
- moved D4 39.4 mm to (150.2, 90.9), turned to 360 degrees
- moved U1 31.7 mm to (47.9, 92.2)
- moved D1 27.3 mm to (152.7, 65.5), turned to 540 degrees
- moved D2 24.8 mm to (150.2, 62.9)
- moved D3 20.1 mm to (152.7, 88.3)
Connections:
- removed net U2_2A: U2.7, U3.2
- removed net U2_3A: U2.10, U3.12
- new net U1_A1: PIR1.1, U1.A1
- new net U1_A2: PIR2.1, U1.A2
- new net U1_D11: U1.D11, U3.7
- new net U1_D12: U1.D12, U3.9
- net M1_+: now also D1.2, D2.1, U3.11; no longer D2.2, D4.1, U2.6
- net M1_-: now also D3.2, D4.1, U3.14; no longer D1.2, D3.1, U2.3
- net M2_+: now also D5.2, D7.1, U3.3; no longer D6.1, D8.2, U2.11
- net M2_-: now also D6.2, D8.1, U3.6; no longer D5.2, D9.1, U2.14
- net U1_5V: now also D2.2, D7.2, D8.2, PIR1.2, PIR2.2, U2.3, U3.16, U3.8; no longer D3.2, D6.2, D9.2, U2.16, U2.8, U3.14, U5.3
- net U1_A0: now also U2.1; no longer U5.2
- net U1_D10: now also U3.1; no longer U2.1
- net U1_D3: now also U3.15; no longer U2.15, U3.13
- net U1_D7: now also U3.2; no longer U2.2, U3.1
- net U1_D9: now also U3.10; no longer U2.9
- net U1_GND: now also D3.1, D6.1, PIR1.3, PIR2.3, U2.2, U3.12, U3.13, U3.4, U3.5; no longer D2.1, D8.1, U2.12, U2.13, U2.4, U2.5, U3.7, U5.1
Other:
- board size 259.3 x 146.3 mm -> 204.1 x 166.8 mm
